File: electronics/amplifier/amplifier.kicad_pcb (KiCad board)
At the start: 2 copper layers, 160 x 100 mm, 107 parts, among them K1 FRT5_separated, K2 FRT5_separated, K4 screw_terminal_2x01, K5 screw_terminal_2x01, P1 CONN_02X01, P2 CONN_02X01, P3 CONN_01X01, P4 CONN_02X01, P5 CONN_01X03, Q1 BC548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

Commit message: added 3dmodels etc.
Parts:
- R34: footprint Resistors_ThroughHole:Resistor_Vertical_RM5mm -> special_symbols:Resistor_Vertical_RM2.5mm
- moved RL1 130.8 mm to (85.3, 95.5)
- moved K1 127.2 mm to (100.3, 95.5)
- moved R34 1.27 mm to (204.5, 50.0)
Routing:
- net Net-(C29-Pad1): track 3.09 -> 5.59 mm
- net +24V: track 200.9 -> 201.4 mm, vias 1 -> 2
Changed lines of the file:
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@@
   (general
     (links 181)
-    (no_connects 125)
-    (area 0 0 0 0)
+    (no_connects 124)
+    (area -7.895001 -140.365 441.393001 161.603)
     (thickness 1.6)
     (drawings 0)
-    (tracks 144)
+    (tracks 149)
     (zones 0)
     (modules 107)
@@
   )
   (module special_symbols:Relay_DPDT_FRT5 (layer F.Cu)
-    (at 69.85 -27.94)
+    (at 100.33 95.504)
     (descr "IM Signal Relay, DPDT, FRT5, narrow footprint")
     (tags "Relay DPDT IM-relay FRT5")
@@
   )
   (module special_symbols:Relay_SPDT_HJR-4102 (layer F.Cu)
-    (at 35.56 -25.4)
+    (at 85.344 95.504)
     (descr "IM Signal Relay, SPDT, HJR-4102")
     (tags "Relay SPDT IM-relay HJR-4102")
@@
   )
   (module Resistors_ThroughHole:Resistor_Vertical_RM5mm (layer F.Cu)
-    (at 204.47 51.308 270)
-    (descr "Resistor, Vertical, RM 5mm, 1/3W,")
-    (tags "Resistor, Vertical, RM 5mm, 1/3W,")
-    (fp_text reference R34 (at 2.70002 -3.29946 270) (layer F.SilkS)
-      (effects (font (size 1 1) (thickness 0.15)))
-    )
-    (fp_text value 2k2 (at 0 4.50088 270) (layer F.Fab)
-      (effects (font (size 1 1) (thickness 0.15)))
-    )
-    (fp_line (start -0.09906 0) (end 0.9017 0) (layer F.SilkS) (width 0.15))
-    (fp_circle (center -2.49936 0) (end 0 0) (layer F.SilkS) (width 0.15))
-    (pad 1 thru_hole circle (at -2.49936 0 270) (size 1.99898 1.99898) (drill 1.00076) (layers *.Cu *.SilkS *.Mask)
-      (net 32 "Net-(C30-Pad1)"))
-    (pad 2 thru_hole circle (at 2.5019 0 270) (size 1.99898 1.99898) (drill 1.00076) (layers *.Cu *.SilkS *.Mask)
-      (net 31 "Net-(C29-Pad1)"))
-  )
-  (module Resistors_ThroughHole:Resistor_Vertical_RM5mm (layer F.Cu)
     (at 140.97 41.402)
     (descr "Resistor, Vertical, RM 5mm, 1/3W,")
@@
     (pad "" np_thru_hole circle (at 5.00126 -5.00126 180) (size 3.50012 3.50012) (drill 3.50012) (layers *.Cu *.Mask F.SilkS))
   )
+  (module special_symbols:Resistor_Vertical_RM2.5mm (layer F.Cu)
+    (at 204.47 50.038 270)
+    (descr "Resistor, Vertical, RM 2.5mm,")
+    (tags "Resistor, Vertical, RM 2.5mm,")
+    (fp_text reference R34 (at 0 -2.032 270) (layer F.SilkS)
+      (effects (font (size 1 1) (thickness 0.15)))
+    )
+    (fp_text value 2k2 (at 0 2.032 270) (layer F.Fab)
+      (effects (font (size 1 1) (thickness 0.15)))
+    )
+    (fp_circle (center -1.27 0) (end -1.016 1.27) (layer F.SilkS) (width 0.15))
+    (fp_line (start 1.27 0) (end -1.27 0) (layer F.SilkS) (width 0.15))
+    (pad 1 thru_hole circle (at -1.27 0 270) (size 1.99898 1.99898) (drill 1.00076) (layers *.Cu *.SilkS *.Mask)
+      (net 32 "Net-(C30-Pad1)"))
+    (pad 2 thru_hole circle (at 1.27 0 270) (size 1.99898 1.99898) (drill 1.00076) (layers *.Cu *.SilkS *.Mask)
+      (net 31 "Net-(C29-Pad1)"))
+    (model ../Resistor_Vertical_RM2_5mm.wrl
+      (at (xyz 0.05 0 0))
+      (scale (xyz 0.395 0.395 0.395))
+      (rotate (xyz 0.395 90 0))
+    )
+  )
   (segment (start 153.67 76.2) (end 153.67 71.374) (width 0.7) (layer B.Cu) (net 1))
   (segment (start 146.35988 64.06388) (end 146.35988 44.43984) (width 0.7) (layer B.Cu) (net 1))
@@
   (segment (start 204.47 61.896) (end 204.47 66.802) (width 0.7) (layer B.Cu) (net 4))
   (segment (start 143.002 77.978) (end 143.002 74.93) (width 0.7) (layer B.Cu) (net 5))
+  (via (at 195.58 46.736) (size 1) (drill 0.4) (layers F.Cu B.Cu) (net 6))
+  (segment (start 195.58 46.736) (end 195.58 46.482) (width 0.7) (layer F.Cu) (net 6))
+  (segment (start 195.58 46.482) (end 195.326 46.482) (width 0.7) (layer F.Cu) (net 6))
+  (segment (start 195.326 46.482) (end 195.58 46.482) (width 0.7) (layer F.Cu) (net 6))
   (via (at 195.58 37.846) (size 1) (drill 0.4) (layers F.Cu B.Cu) (net 6))
-  (segment (start 171.45 43.942) (end 177.546 37.846) (width 2) (layer B.Cu) (net 6))
-  (segment (start 177.546 37.846) (end 195.58 37.846) (width 2) (layer B.Cu) (net 6))
-  (segment (start 171.45 46.99) (end 171.45 43.942) (width 2) (layer B.Cu) (net 6))
-  (segment (start 195.58 39.37) (end 195.58 46.736) (width 2) (layer F.Cu) (net 6))
   (segment (start 195.58 37.846) (end 195.58 39.37) (width 2) (layer F.Cu) (net 6))
+  (segment (start 195.58 39.37) (end 195.58 46.482) (width 2) (layer F.Cu) (net 6))
+  (segment (start 171.45 46.99) (end 171.45 43.942) (width 2) (layer B.Cu) (net 6))
+  (segment (start 177.546 37.846) (end 195.58 37.846) (width 2) (layer B.Cu) (net 6))
+  (segment (start 171.45 43.942) (end 177.546 37.846) (width 2) (layer B.Cu) (net 6))
   (segment (start 198.882 104.728) (end 201.756 104.728) (width 1) (layer B.Cu) (net 6))
   (segment (start 201.756 104.728) (end 203.454 106.426) (width 1) (layer B.Cu) (net 6))
@@
   (segment (start 182.88 62.23) (end 184.404 62.23) (width 0.7) (layer B.Cu) (net 30))
   (segment (start 184.404 62.23) (end 186.436 60.198) (width 0.7) (layer B.Cu) (net 30))
-  (segment (start 204.47 56.896) (end 204.47 53.8099) (width 0.7) (layer B.Cu) (net 31))
+  (segment (start 204.47 51.308) (end 204.47 53.8099) (width 0.7) (layer B.Cu) (net 31))
+  (segment (start 204.47 53.8099) (end 204.47 56.896) (width 0.7) (layer B.Cu) (net 31))
   (segment (start 193.04 83.82) (end 193.04 79.756) (width 2) (layer B.Cu) (net 32))
   (segment (start 199.898 52.324) (end 199.898 48.80864) (width 2) (layer B.Cu) (net 32))

Commit message: diverse libs
Parts:
- moved P5 160.0 mm to (96.3, 127.8)
- moved K2 84.9 mm to (81.8, 70.4)
- moved RL1 42.3 mm to (81.8, 53.3)
- moved K1 20.9 mm to (81.5, 86.4)
- moved U6 17.3 mm to (173.7, 132.6)
- moved U4 17.0 mm to (157.2, 132.3)

Commit message: finished amplifier PCB
Parts:
- removed K5: screw_terminal_2x01, Connect:bornier2
- removed Q2, Q3: BC548, TO_SOT_Packages_THT:TO-92_Molded_Narrow
- removed R19, R20: 220R, Resistors_ThroughHole:Resistor_Horizontal_RM10mm
- removed REF**: EuroBoard160mmX100mm_holes, EuroBoard_Outline:EuroBoard160mmX100mm_holes
- removed W1, W10, W11, W2, W3, W4, W5, W6, W7, W8, W9: TEST_1P, Pin_Headers:Pin_Header_Straight_1x01
- added C33: 2200µF, Capacitors_ThroughHole:C_Radial_D30_L51_P10, F.Cu at (58.9, 67.1)
- added C34: 2200µF, Capacitors_ThroughHole:C_Radial_D30_L51_P10, F.Cu at (90.0, 67.3)
- added C35: 2200µF, Capacitors_ThroughHole:C_Radial_D30_L51_P10, F.Cu at (58.9, 99.2)
- added C36: 100nF, Capacitors_ThroughHole:C_Disc_D6_P5, F.Cu at (79.5, 86.2)
- added H1: screw_terminal_2x01, Connect:bornier2, F.Cu at (42.2, 44.7)
- added H2: screw_terminal_2x01, Connect:bornier2, F.Cu at (79.2, 119.1)
- C13: value 100nF -> 100µF; footprint Capacitors_ThroughHole:C_Disc_D7.5_P5 -> Capacitors_ThroughHole:C_Radial_D6.3_L11.2_P2.5
- C15: footprint Capacitors_ThroughHole:C_Radial_D10_L13_P5 -> Capacitors_ThroughHole:C_Radial_D6.3_L11.2_P2.5
- D2: value LED -> Diode_Bridge; footprint LEDs:LED-5MM -> special_symbols:Diode_Bridge_32x5.7
- P3: value CONN_01X01 -> CONN_02X01; footprint Pin_Headers:Pin_Header_Straight_1x01 -> Pin_Headers:Pin_Header_Straight_2x01
- R13, R27, R4, R8: footprint Resistors_ThroughHole:Resistor_Horizontal_RM10mm -> special_symbols:Resistor_Vertical_RM2.5mm
- R16: value 10k -> 1R; footprint Resistors_ThroughHole:Resistor_Horizontal_RM10mm -> Resistors_ThroughHole:Resistor_Ceramic_Horizontal_L23mm-W9mm-H9mm-p30mm
- R17: value 10k -> 1k5; footprint Resistors_ThroughHole:Resistor_Horizontal_RM10mm -> Resistors_ThroughHole:Resistor_Horizontal_RM15mm
- R5: footprint Resistors_ThroughHole:Resistor_Vertical_RM5mm -> special_symbols:Resistor_Vertical_RM2.5mm
- U5: value 74HC04 -> LM7805CT; footprint Housings_DIP:DIP-14_W7.62mm_LongPads -> TO-220
- moved R27 319.1 mm to (133.3, 116.3)
- moved R7 317.8 mm to (109.2, 118.9)
- moved C8 311.0 mm to (126.0, 102.6)
- moved R23 310.3 mm to (142.2, 118.9), turned to 180 degrees
- moved R21 310.1 mm to (137.2, 106.2), turned to 270 degrees
- moved U2 307.2 mm to (121.9, 113.8)
- moved C22 301.9 mm to (123.4, 108.7)
- moved C20 295.0 mm to (146.3, 118.9)
- moved R8 291.5 mm to (118.1, 121.4)
- moved R9 291.4 mm to (109.2, 116.3)
- moved C11 272.4 mm to (111.8, 106.2)
- moved R17 265.7 mm to (81.8, 112.1), turned to 90 degrees
- moved C17 265.6 mm to (132.6, 125.5)
- moved R16 257.8 mm to (90.0, 102.0), turned to 90 degrees
- moved C19 253.7 mm to (193.0, 106.7), turned to 180 degrees
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Connections:
- C13 pad 1: GND -> +5V
- C13 pad 2: +15V -> GND
- C31 pad 2: +5V -> +24V
- D2 pad 1: Net-(D2-Pad1) -> Net-(C33-Pad2)
- D3 pad 1: Net-(D3-Pad1) -> Net-(C33-Pad2)
- P1 pad 1: Net-(P1-Pad1) -> RELAIS
- P2 pad 1: Net-(P1-Pad1) -> Net-(P2-Pad1)
- P2 pad 2: Net-(P2-Pad2) -> RELAIS
- P3 pad 1: Net-(P1-Pad1) -> RELAIS
- P4 pad 1: Net-(P1-Pad1) -> Net-(P4-Pad1)
- P4 pad 2: Net-(P4-Pad2) -> RELAIS
- R15 pad 2: Net-(R15-Pad2) -> Net-(P2-Pad1)
- R16 pad 1: Net-(Q2-Pad2) -> Net-(H2-Pad2)
- R16 pad 2: Net-(R16-Pad2) -> Net-(C33-Pad1)
- R17 pad 1: Net-(Q3-Pad2) -> Net-(H2-Pad2)
- R17 pad 2: Net-(R17-Pad2) -> Net-(D3-Pad2)
- R18 pad 2: Net-(R18-Pad2) -> Net-(P4-Pad1)
- R35 pad 2: Net-(R35-Pad2) -> Net-(P1-Pad2)
- U5 pad 1: Net-(P1-Pad1) -> +24V
- U5 pad 2: Net-(R15-Pad2) -> GND
- U5 pad 3: Net-(P1-Pad1) -> +5V
Routing:
- net GND: track 250.3 -> 639.4 mm, vias 2 -> 4
- net Net-(C33-Pad2): track 0.00 -> 164.6 mm
- net +5V: track 0.00 -> 155.5 mm, vias 0 -> 6
- net +15V: track 8.42 -> 153.1 mm
- net Net-(C33-Pad1): track 0.00 -> 124.5 mm
- net +24V: track 201.4 -> 279.6 mm
- net VPP: track 0.00 -> 68.8 mm, vias 0 -> 4
- net Net-(K2-Pad7): track 0.00 -> 67.8 mm
- net Net-(P1-Pad2): track 0.00 -> 64.8 mm, vias 0 -> 2
- net Net-(K1-Pad7): track 0.00 -> 60.5 mm
- net Net-(C17-Pad2): track 0.00 -> 58.9 mm, vias 0 -> 2
- net Net-(K2-Pad9): track 0.00 -> 56.5 mm, vias 0 -> 2
- net Net-(D2-Pad2): track 0.00 -> 48.3 mm
- net Net-(K1-Pad9): track 0.00 -> 40.8 mm
- net Net-(C19-Pad2): track 0.00 -> 33.5 mm
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Other:
- board size 160 x 100 mm -> 170.9 x 93.2 mm

Commit message: changed some parts
Parts:
- C33, C34, C35: footprint Capacitors_ThroughHole:C_Radial_D30_L51_P10 -> special_symbols:C_Radial_D30_L51_P10_3pin
- D2: value Diode_Bridge -> B40C5000
- R16: footprint Resistors_ThroughHole:Resistor_Ceramic_Horizontal_L23mm-W9mm-H9mm-p30mm -> special_symbols:Resistor_Ceramic_Horizontal_L25mm-W6.4mm-H6.4mm-p30mm
- moved R16 0.40 mm to (89.9, 101.6)
Routing:
- net Net-(C33-Pad2): track 164.6 -> 168.8 mm
- net Net-(C33-Pad1): track 124.5 -> 121.2 mm
